File: 5wayjoy.kicad_pcb (KiCad board)
At the start: 2 copper layers, 36.9 x 15.7 mm, 6 parts, among them J1 Conn_01x04_Socket, U2 MCP23008-xSS

Commit message: more files
Parts:
- added R5: 0, Resistor_SMD:R_0805_2012Metric_Pad1.20x1.40mm_HandSolder, B.Cu at (175.8, 83.9)
Routing:
- net VCC: track 29.3 -> 31.9 mm
Other:
- board size 36.9 x 15.7 mm -> 36.9 x 20.6 mm
